Commit message: gripbot2

File: urdf/gripbot.urdf (robot description, URDF)
Before this commit: robot gripbot, 5 links, 4 joints
Links:
- link arm_visual_link: mass 0.10 -> 19.56717
- link base_column_link: mass 0.7 -> 33.204
- link base_mount_link: mass 3.7 -> 240
- link forearm_visual_link: mass 0.06 -> 9.055067
- link girdle_visual_link: mass 0.4 -> 8.62636
