Commit message: blend

File: urdf/gripbot_2.urdf (robot description, URDF)
Before this commit: robot gripbot, 16 links, 16 joints
Links:
- removed link new_link
- added link finger_3_distal_link, mass 0.101; collision box size=0.0175 0.02023 0.04043; visual mesh filename=package://gripbot_description/meshes/stl/FingerDistal.stl scale=1.0 1.0 1.0
- added link finger_3_mid_link, mass 0.101; collision box size=0.01784 0.01899 0.03281; visual mesh filename=package://gripbot_description/meshes/stl/Cube.016.stl scale=1.0 1.0 1.0
- link arm_visual_link: mass 1.0 -> 19.56717; geometry collision box size=0.15244 0.53451 0.15245; collision box size=0.18304 0.15204 0.15204
- link base_column_link: mass 40.0 -> 33.204; geometry collision box size=0.15423 0.15423 0.30549; collision box size=0.15655 0.17927 0.17927
- link base_mount_link: mass 120.0 -> 240
- link base_wrist_link: mass None -> 3.6; geometry collision box size=0.1135 0.07446 0.07319; collision cylinder length=0.074303 radius=0.04771
- link finger_1_base_link: mass None -> 0.1010; geometry collision cylinder length=0.034775 radius=0.010094; visual mesh filename=package://gripbot_description/meshes/stl/FingerBase.stl scale=1.0 1.0 1.0
- link finger_1_distal_link: mass None -> 0.101
- link finger_1_mid_link: mass None -> 0.101
- link finger_1_proximal_link: mass None -> 0.101; geometry collision box size=0.01754 0.01751 0.05287; visual mesh filename=package://gripbot_description/meshes/stl/FingerProximal.001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 scale=1.0 1.0 1.0
- link finger_2_base_link: mass None -> 0.101; geometry collision cylinder length=0.034775 radius=0.010094; visual mesh filename=package://gripbot_description/meshes/stl/FingerBase.001.stl scale=1.0 1.0 1.0
- link finger_2_distal_link: mass None -> 0.101
- link finger_2_mid_link: mass None -> 0.101
- link finger_2_proximal_link: mass None -> 0.101
- link finger_3_proximal_link: mass None -> 0.101; geometry collision box size=0.01755 0.01858 0.05311; collision box size=0.03477 0.02019 0.02019
- link forearm_visual_link: mass 1.0 -> 9.055067
- link girdle_visual_link: mass 3.0 -> 8.62636; geometry collision box size=0.15423 0.15423 0.30864; visual mesh filename=package://gripbot_description/meshes/stl/Circle.001.stl scale=1.0 1.0 1.0
Joints:
- joint base_wrist_link: limit lower=-3.14159 upper=3.14159 effort=10000.0 velocity=0 -> lower=-3.14159 upper=3.14159 effort=10000.0 velocity=6.00
- joint finger_1_base_link: limit lower=-2.04204 upper=0.7854 effort=10000.0 velocity=0 -> lower=-2.04204 upper=0.7854 effort=10000.0 velocity=60000
- joint finger_1_distal_link: limit lower=0 upper=1.5708 effort=10000.0 velocity=0 -> lower=0 upper=1.5708 effort=10000.0 velocity=60000
- joint finger_1_mid_link: limit lower=0 upper=1.5708 effort=10000.0 velocity=0 -> lower=0 upper=1.5708 effort=10000.0 velocity=60000
- joint finger_1_proximal_link: limit lower=0 upper=1.5708 effort=10000.0 velocity=0 -> lower=0 upper=1.5708 effort=10000.0 velocity=60000
- joint finger_2_base_link: limit lower=-0.7854 upper=1.72788 effort=10000.0 velocity=0 -> lower=-0.7854 upper=1.72788 effort=10000.0 velocity=60000
- joint finger_2_distal_link: limit lower=-1.5708 upper=0 effort=10000.0 velocity=0 -> lower=-1.5708 upper=0 effort=10000.0 velocity=60000
- joint finger_2_mid_link: limit lower=-1.5708 upper=0 effort=10000.0 velocity=0 -> lower=-1.5708 upper=0 effort=10000.0 velocity=60000; parent new_link -> finger_2_proximal_link
- joint finger_2_proximal_link: child new_link -> finger_2_proximal_link; limit lower=0 upper=1.5708 effort=10000.0 velocity=0 -> lower=0 upper=1.5708 effort=10000.0 velocity=60000; origin xyz=0 -0.00041 0.04213 rpy=0 0 0 -> xyz=0 0 0 rpy=0 0 0
- joint finger_3_distal_link: child new_link -> finger_3_distal_link; limit lower=0 upper=1.72788 effort=10000.0 velocity=0 -> lower=0 upper=1.72788 effort=10000.0 velocity=60000; origin xyz=0 -0.00041 0.04213 rpy=0 0 0 -> xyz=0 -0.00041 0.04199 rpy=0 0 0; parent new_link -> finger_3_mid_link
- joint finger_3_mid_link: child new_link -> finger_3_mid_link; limit lower=0 upper=1.72788 effort=10000.0 velocity=0 -> lower=0 upper=1.72788 effort=10000.0 velocity=60000; origin xyz=0 -0.00041 0.04213 rpy=0 0 0 -> xyz=0 -0.00041 0.06051 rpy=0 0 0
- joint finger_3_proximal_link: limit lower=-0.7854 upper=1.72788 effort=10000.0 velocity=0 -> lower=-0.7854 upper=1.72788 effort=10000.0 velocity=60000
- joint forearm_visual_link: limit lower=-1.5708 upper=2.18166 effort=135.0 velocity=6.28319 -> lower=-1.5708 upper=2.18166 effort=135.0 velocity=60000.28319

Commit message: initial

File: urdf/gripbot_2.urdf (robot description, URDF)
Before this commit: robot gripbot, 17 links, 16 joints
Links:
- added link dummy_link
Joints:
- added joint dummy_joint: type fixed, parent dummy_link, child base_mount_link

Commit message: Working controlls

File: urdf/gripbot_2.urdf (robot description, URDF)
Before this commit: robot gripbot, 18 links, 17 joints
Joints:
- joint base_wrist_link: limit lower=-3.14159 upper=3.14159 effort=10000.0 velocity=6.00 -> lower=-1.5708 upper=1.5708 effort=10000.0 velocity=6.00
- joint finger_2_base_link: limit lower=-0.7854 upper=1.72788 effort=10000.0 velocity=60000 -> lower=-0.7854 upper=2.04204 effort=10000.0 velocity=60000
- joint finger_2_proximal_link: limit lower=0 upper=1.5708 effort=10000.0 velocity=60000 -> lower=-1.5708 upper=0 effort=10000.0 velocity=60000
